File: SOIC16_Breakout_Boards/SOIC_16_Breakout_Board.kicad_sch (KiCad schematic)
At the start: 6 parts, among them J1 Conn_01x08, J2 Conn_01x08, J3 Conn_01x01, J4 Conn_01x01

Commit message: Created PCB designs for the 14, 16 & 20 pic SOIC's
Finalized and committed pcb designs for the 14, 16, and 20 SOIC breakout boards
Parts:
- J1, J2: footprint (none) -> Connector_PinSocket_2.54mm:PinSocket_1x08_P2.54mm_Vertical
- SOIC1: footprint (none) -> SOIC_Footprints:16_Pin_SOIC_Board
Connections:
- net at J2.1 (Pin_1): now also SOIC1.16; no longer SOIC1.9
- net at J2.2 (Pin_2): now also SOIC1.15; no longer SOIC1.10
- net at J2.3 (Pin_3): now also SOIC1.14; no longer SOIC1.11
- net at J2.4 (Pin_4): now also SOIC1.13; no longer SOIC1.12
- net at J2.5 (Pin_5): now also SOIC1.12; no longer SOIC1.13
- net at J2.6 (Pin_6): now also SOIC1.11; no longer SOIC1.14
- net at J2.7 (Pin_7): now also SOIC1.10; no longer SOIC1.15
- net at J2.8 (Pin_8): now also SOIC1.9; no longer SOIC1.16
Other:
- moved on the sheet: J1, J2, J3, J4, R1
Changed lines of the file:
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@@
     (rev "0")
   )
-  (wire (pts (xy 123.19 64.77) (xy 125.73 64.77))
+  (wire (pts (xy 132.08 85.09) (xy 134.62 85.09))
     (stroke (width 0) (type default) (color 0 0 0 0))
   )
-  (wire (pts (xy 133.35 64.77) (xy 135.89 64.77))
+  (wire (pts (xy 142.24 85.09) (xy 144.78 85.09))
     (stroke (width 0) (type default) (color 0 0 0 0))
   )
-  (symbol (lib_id "Connector_Generic:Conn_01x01") (at 140.97 64.77 0) (unit 1)
+  (symbol (lib_id "Connector_Generic:Conn_01x01") (at 149.86 85.09 0) (unit 1)
     (in_bom yes) (on_board yes)
-    (property "Reference" "J4" (id 0) (at 140.97 59.69 0))
-    (property "Value" "Conn_01x01" (id 1) (at 140.97 62.23 0))
-    (property "Footprint" "Connector_PinSocket_2.54mm:PinSocket_1x01_P2.54mm_Vertical" (id 2) (at 140.97 64.77 0)
+    (property "Reference" "J4" (id 0) (at 149.86 80.01 0))
+    (property "Value" "Conn_01x01" (id 1) (at 149.86 82.55 0))
+    (property "Footprint" "Connector_PinSocket_2.54mm:PinSocket_1x01_P2.54mm_Vertical" (id 2) (at 149.86 85.09 0)
       (effects (font (size 1.27 1.27)) hide)
     )
-    (property "Datasheet" "~" (id 3) (at 140.97 64.77 0)
+    (property "Datasheet" "~" (id 3) (at 149.86 85.09 0)
       (effects (font (size 1.27 1.27)) hide)
     )
     (pin "1")
   )
-  (symbol (lib_id "Connector_Generic:Conn_01x01") (at 118.11 64.77 0) (mirror y) (unit 1)
+  (symbol (lib_id "Connector_Generic:Conn_01x01") (at 127 85.09 0) (mirror y) (unit 1)
     (in_bom yes) (on_board yes)
-    (property "Reference" "J3" (id 0) (at 119.38 59.69 0)
+    (property "Reference" "J3" (id 0) (at 128.27 80.01 0)
       (effects (font (size 1.27 1.27)) (justify left))
     )
-    (property "Value" "Conn_01x01" (id 1) (at 123.19 62.23 0)
+    (property "Value" "Conn_01x01" (id 1) (at 132.08 82.55 0)
       (effects (font (size 1.27 1.27)) (justify left))
     )
-    (property "Footprint" "Connector_PinSocket_2.54mm:PinSocket_1x01_P2.54mm_Vertical" (id 2) (at 118.11 64.77 0)
+    (property "Footprint" "Connector_PinSocket_2.54mm:PinSocket_1x01_P2.54mm_Vertical" (id 2) (at 127 85.09 0)
       (effects (font (size 1.27 1.27)) hide)
     )
-    (property "Datasheet" "~" (id 3) (at 118.11 64.77 0)
+    (property "Datasheet" "~" (id 3) (at 127 85.09 0)
       (effects (font (size 1.27 1.27)) hide)
     )
     (pin "1")
   )
-  (symbol (lib_id "Connector_Generic:Conn_01x08") (at 142.24 76.2 0) (unit 1)
+  (symbol (lib_id "Connector_Generic:Conn_01x08") (at 151.13 96.52 0) (unit 1)
     (in_bom yes) (on_board yes)
-    (property "Reference" "J2" (id 0) (at 147.32 81.28 90)
+    (property "Reference" "J2" (id 0) (at 156.21 101.6 90)
       (effects (font (size 1.27 1.27)) (justify left))
     )
-    (property "Value" "Conn_01x08" (id 1) (at 144.78 81.28 90)
+    (property "Value" "Conn_01x08" (id 1) (at 153.67 101.6 90)
       (effects (font (size 1.27 1.27)) (justify left))
     )
-    (property "Footprint" "" (id 2) (at 142.24 76.2 0)
+    (property "Footprint" "Connector_PinSocket_2.54mm:PinSocket_1x08_P2.54mm_Vertical" (id 2) (at 151.13 96.52 0)
       (effects (font (size 1.27 1.27)) hide)
     )
-    (property "Datasheet" "~" (id 3) (at 142.24 76.2 0)
+    (property "Datasheet" "~" (id 3) (at 151.13 96.52 0)
       (effects (font (size 1.27 1.27)) hide)
     )
@@
     (pin "8")
   )
-  (symbol (lib_id "Connector_Generic:Conn_01x08") (at 116.84 76.2 0) (mirror y) (unit 1)
+  (symbol (lib_id "Connector_Generic:Conn_01x08") (at 125.73 96.52 0) (mirror y) (unit 1)
     (in_bom yes) (on_board yes)
-    (property "Reference" "J1" (id 0) (at 111.76 76.2 90))
-    (property "Value" "Conn_01x08" (id 1) (at 114.3 76.2 90))
-    (property "Footprint" "" (id 2) (at 116.84 76.2 0)
+    (property "Reference" "J1" (id 0) (at 120.65 96.52 90))
+    (property "Value" "Conn_01x08" (id 1) (at 123.19 96.52 90))
+    (property "Footprint" "Connector_PinSocket_2.54mm:PinSocket_1x08_P2.54mm_Vertical" (id 2) (at 125.73 96.52 0)
       (effects (font (size 1.27 1.27)) hide)
     )
-    (property "Datasheet" "~" (id 3) (at 116.84 76.2 0)
+    (property "Datasheet" "~" (id 3) (at 125.73 96.52 0)
       (effects (font (size 1.27 1.27)) hide)
     )
@@
     (pin "8")
   )
-  (symbol (lib_id "8_Pin_SOIC_Board:16_Pin_SOIC_Board") (at 129.54 76.2 0) (unit 1)
+  (symbol (lib_id "8_Pin_SOIC_Board:16_Pin_SOIC_Board") (at 138.43 96.52 0) (unit 1)
     (in_bom yes) (on_board yes)
-    (property "Reference" "SOIC1" (id 0) (at 129.54 91.44 0))
-    (property "Value" "16_Pin_SOIC_Board" (id 1) (at 129.54 88.9 0))
-    (property "Footprint" "" (id 2) (at 129.54 76.2 0)
+    (property "Reference" "SOIC1" (id 0) (at 138.43 109.22 0))
+    (property "Value" "16_Pin_SOIC_Board" (id 1) (at 138.43 111.76 0))
+    (property "Footprint" "SOIC_Footprints:16_Pin_SOIC_Board" (id 2) (at 138.43 96.52 0)
       (effects (font (size 1.27 1.27)) hide)
     )
-    (property "Datasheet" "" (id 3) (at 129.54 76.2 0)
+    (property "Datasheet" "" (id 3) (at 138.43 96.52 0)
       (effects (font (size 1.27 1.27)) hide)
     )
@@
     (pin "9")
   )
-  (symbol (lib_id "Device:R_US") (at 129.54 64.77 270) (unit 1)
+  (symbol (lib_id "Device:R_US") (at 138.43 85.09 270) (unit 1)
     (in_bom yes) (on_board yes) (fields_autoplaced)
-    (property "Reference" "R1" (id 0) (at 129.54 58.42 90))
-    (property "Value" "R_US" (id 1) (at 129.54 60.96 90))
-    (property "Footprint" "Resistor_SMD:R_0805_2012Metric" (id 2) (at 129.286 65.786 90)
+    (property "Reference" "R1" (id 0) (at 138.43 78.74 90))
+    (property "Value" "R_US" (id 1) (at 138.43 81.28 90))
+    (property "Footprint" "Resistor_SMD:R_0805_2012Metric" (id 2) (at 138.176 86.106 90)
       (effects (font (size 1.27 1.27)) hide)
     )
-    (property "Datasheet" "~" (id 3) (at 129.54 64.77 0)
+    (property "Datasheet" "~" (id 3) (at 138.43 85.09 0)
       (effects (font (size 1.27 1.27)) hide)
     )
@@
   (symbol_instances
     (path "/ad79c9d2-02bc-460f-b8b4-643b28873af7"
-      (reference "J1") (unit 1) (value "Conn_01x08") (footprint "")
+      (reference "J1") (unit 1) (value "Conn_01x08") (footprint "Connector_PinSocket_2.54mm:PinSocket_1x08_P2.54mm_Vertical")
     )
     (path "/840f91ee-4e9a-470c-a7d7-94ae66d50398"
-      (reference "J2") (unit 1) (value "Conn_01x08") (footprint "")
+      (reference "J2") (unit 1) (value "Conn_01x08") (footprint "Connector_PinSocket_2.54mm:PinSocket_1x08_P2.54mm_Vertical")
     )
     (path "/7dfc8e4d-cb13-4be6-bcf8-32029bab029b"
@@
       (reference "R1") (unit 1) (value "R_US") (footprint "Resistor_SMD:R_0805_2012Metric")
     )
-    (path "/e982189f-ef9a-4f4a-8f00-086ac9174a75"
-      (reference "SOIC1") (unit 1) (value "16_Pin_SOIC_Board") (footprint "")
+    (path "/c45af6d6-304b-4e86-af6c-0314de02283d"
+      (reference "SOIC1") (unit 1) (value "16_Pin_SOIC_Board") (footprint "SOIC_Footprints:16_Pin_SOIC_Board")
     )
   )
